Commit message: Part 1: the centre is shut by the TORSO, not by the wearer's arms
The project's answer to "why can the work not be in the centre" has been the
wearer's own forearm, measured against a mannequin whose arms hang rigidly at
its sides. That is a modelling choice, so the posture is now a variable with
one source and the sweep was re-run in four postures plus the limit case of no
arms at all.

The centre does not open in any of them. With the wearer's arms deleted
entirely, min |x| is still 0.300 (left) and 0.375 (right), every column from
0.125 to 0.300 binds on the TORSO, and at |x| = 0.10 the clearance is -0.007
and -0.013 m, which is the arm inside the person's chest. Holding the arms
clear is worth 25 mm on the left and 75 mm on the right.

Folding the arms across the chest costs 75 mm. Clasping them behind the back
or holding them out to the sides puts the wearer's own limbs inside the
BACK-mounted robot's envelope and breaches the 150 mm floor at the HOME pose,
before anything has been asked of the arm. The useful instruction to a wearer
is "arms down at your sides", which is what the model already assumed and what
nobody had checked was the best of the options.

base_link caps every clearance figure at 0.1610 m. It is a link no joint moves,
so a reading of exactly 0.1610 is the mount's clearance and not the arm's, and
the 150 mm floor has 11 mm of headroom before the arm does anything.

Two live instrument faults found on the way:

  clearance.py, which ik_follower_node, real_homing_node and sim_to_real_bridge
  enforce at runtime, modelled a torso, a head and a pair of hips. The wearer's
  arms were not in it, and they are what binds the right arm inboard, so the
  planner's wearer and the follower's wearer were different people.

  record_verification.py drew the wearer's upper arms 150 mm and forearms
  130 mm below where they are, and omitted the hands.

The published innermost-safe columns are stale. centre_vs_height.json records
0.425 / 0.400; re-running that same script unchanged at z = 1.120 returns
0.325 / 0.450 today, matching the new sweep, because the home change moved the
IK seed and therefore the null-space branch. TASK_SPEC is corrected.

Two of my own controls were wrong and both are recorded in findings.md: a
control whose ground truth moves with the thing under test refused two of the
postures the sweep exists to measure, and a malformed shell line left two
stacks running so one measurement read the wrong robot_description. The URDF
control caught that, which is what it is for.

Tests: 545 pass, 2 allowed failures, 0 new.

This commit also lands the previous session's uncommitted work, which was
never checked in: the predictive-avoidance module and its verification, the
centre-on-surface search, the home storage-site audit and the grasp-approach
measurements.

File: src/srl_description/urdf/human_backpack.xacro (robot description, xacro)
@@ -182,60 +182,257 @@
          The previous model had NONE - the render showed a torso with
          only the two Kinova arms, which is why the SRL arms read as the
-         wearer's arms. Upper arm / forearm / hand, hanging at rest,
-         shoulder line z=1.43 matching the top of the chest box. -->
-    <link name="human_left_upper_arm">
-      <collision><geometry><cylinder radius="0.050" length="0.30"/></geometry></collision>
-      <visual><geometry><cylinder radius="0.050" length="0.30"/></geometry>
-        <material name="shirt"/></visual>
-    </link>
-    <joint name="torso_to_human_left_upper_arm" type="fixed">
-      <parent link="torso"/><child link="human_left_upper_arm"/>
-      <origin xyz="0.21 0 0.23" rpy="0 0 0"/>
-    </joint>
-    <link name="human_left_lower_arm">
-      <collision><geometry><cylinder radius="0.045" length="0.26"/></geometry></collision>
-      <visual><geometry><cylinder radius="0.045" length="0.26"/></geometry>
-        <material name="skin"/></visual>
-    </link>
-    <joint name="torso_to_human_left_lower_arm" type="fixed">
-      <parent link="torso"/><child link="human_left_lower_arm"/>
-      <origin xyz="0.21 0 -0.05" rpy="0 0 0"/>
-    </joint>
-    <link name="human_left_hand">
-      <collision><geometry><box size="0.09 0.05 0.18"/></geometry></collision>
-      <visual><geometry><box size="0.09 0.05 0.18"/></geometry>
-        <material name="skin"/></visual>
-    </link>
-    <joint name="torso_to_human_left_hand" type="fixed">
-      <parent link="torso"/><child link="human_left_hand"/>
-      <origin xyz="0.21 0 -0.27" rpy="0 0 0"/>
-    </joint>
-    <link name="human_right_upper_arm">
-      <collision><geometry><cylinder radius="0.050" length="0.30"/></geometry></collision>
-      <visual><geometry><cylinder radius="0.050" length="0.30"/></geometry>
-        <material name="shirt"/></visual>
-    </link>
-    <joint name="torso_to_human_right_upper_arm" type="fixed">
-      <parent link="torso"/><child link="human_right_upper_arm"/>
-      <origin xyz="-0.21 0 0.23" rpy="0 0 0"/>
-    </joint>
-    <link name="human_right_lower_arm">
-      <collision><geometry><cylinder radius="0.045" length="0.26"/></geometry></collision>
-      <visual><geometry><cylinder radius="0.045" length="0.26"/></geometry>
-        <material name="skin"/></visual>
-    </link>
-    <joint name="torso_to_human_right_lower_arm" type="fixed">
-      <parent link="torso"/><child link="human_right_lower_arm"/>
-      <origin xyz="-0.21 0 -0.05" rpy="0 0 0"/>
-    </joint>
-    <link name="human_right_hand">
-      <collision><geometry><box size="0.09 0.05 0.18"/></geometry></collision>
-      <visual><geometry><box size="0.09 0.05 0.18"/></geometry>
-        <material name="skin"/></visual>
-    </link>
-    <joint name="torso_to_human_right_hand" type="fixed">
-      <parent link="torso"/><child link="human_right_hand"/>
-      <origin xyz="-0.21 0 -0.27" rpy="0 0 0"/>
-    </joint>
+         wearer's arms. Upper arm / forearm / hand, shoulder line
+         z=1.43 matching the top of the chest box.
+         THE POSTURE IS A VARIABLE, and the block below is GENERATED.
+         Edit src/srl_teleop/srl_teleop/wearer_posture.py and run
+         scripts/gen_wearer_posture_xacro.py; do not edit it here. The
+         same table feeds mount_guard_node's geometric clearance model,
+         and a posture that reaches one and not the other is a
+         measurement that reports the old answer under a new name. -->
+    <!-- BEGIN GENERATED WEARER ARMS - edit wearer_posture.py, not this -->
+    <!-- Which posture the wearer holds. See wearer_posture.py;
+         SRL_WEARER_ARMS to pick one. -->
+    <xacro:property name="wearer_arms" value="$(optenv SRL_WEARER_ARMS down)"/>
+    <!-- An unknown posture must STOP the build. A typo that silently
+         falls back to the default is a sweep that measures the same
+         wearer five times and reports it as five postures. -->
+    <xacro:unless value="${wearer_arms == 'behind' or wearer_arms == 'down' or wearer_arms == 'folded' or wearer_arms == 'none' or wearer_arms == 'out'}">
+      <!-- a property body is evaluated lazily and would never fire;
+           an attribute is substituted eagerly, so this one does. -->
+      <link name="unknown_wearer_arms_posture_${1/0}"/>
+    </xacro:unless>
+    <xacro:if value="${wearer_arms == 'behind'}">
+      <!-- clasped behind the back, hands crossed at the small of the back -->
+      <link name="human_left_upper_arm">
+        <collision><geometry><cylinder radius="0.05" length="0.3"/></geometry></collision>
+        <visual><geometry><cylinder radius="0.05" length="0.3"/></geometry>
+          <material name="shirt"/></visual>
+      </link>
+      <joint name="torso_to_human_left_upper_arm" type="fixed">
+        <parent link="torso"/><child link="human_left_upper_arm"/>
+        <origin xyz="0.196463 -0.063174 0.244627" rpy="0.434724 -3.04192 0"/>
+      </joint>
+      <link name="human_left_lower_arm">
+        <collision><geometry><cylinder radius="0.045" length="0.26"/></geometry></collision>
+        <visual><geometry><cylinder radius="0.045" length="0.26"/></geometry>
+          <material name="skin"/></visual>
+      </link>
+      <joint name="torso_to_human_left_lower_arm" type="fixed">
+        <parent link="torso"/><child link="human_left_lower_arm"/>
+        <origin xyz="0.0604803 -0.139374 0.067571" rpy="0.100369 -1.89892 0"/>
+      </joint>
+      <link name="human_left_hand">
+        <collision><geometry><box size="0.09 0.05 0.18"/></geometry></collision>
+        <visual><geometry><box size="0.09 0.05 0.18"/></geometry>
+          <material name="skin"/></visual>
+      </link>
+      <joint name="torso_to_human_left_hand" type="fixed">
+        <parent link="torso"/><child link="human_left_hand"/>
+        <origin xyz="-0.116158 -0.170464 -0.0436598" rpy="0.202086 -2.47965 0"/>
+      </joint>
+      <link name="human_right_upper_arm">
+        <collision><geometry><cylinder radius="0.05" length="0.3"/></geometry></collision>
+        <visual><geometry><cylinder radius="0.05" length="0.3"/></geometry>
+          <material name="shirt"/></visual>
+      </link>
+      <joint name="torso_to_human_right_upper_arm" type="fixed">
+        <parent link="torso"/><child link="human_right_upper_arm"/>
+        <origin xyz="-0.196463 -0.063174 0.244627" rpy="0.434724 3.04192 0"/>
+      </joint>
+      <link name="human_right_lower_arm">
+        <collision><geometry><cylinder radius="0.045" length="0.26"/></geometry></collision>
+        <visual><geometry><cylinder radius="0.045" length="0.26"/></geometry>
+          <material name="skin"/></visual>
+      </link>
+      <joint name="torso_to_human_right_lower_arm" type="fixed">
+        <parent link="torso"/><child link="human_right_lower_arm"/>
+        <origin xyz="-0.0604803 -0.139374 0.067571" rpy="0.100369 1.89892 0"/>
+      </joint>
+      <link name="human_right_hand">
+        <collision><geometry><box size="0.09 0.05 0.18"/></geometry></collision>
+        <visual><geometry><box size="0.09 0.05 0.18"/></geometry>
+          <material name="skin"/></visual>
+      </link>
+      <joint name="torso_to_human_right_hand" type="fixed">
+        <parent link="torso"/><child link="human_right_hand"/>
+        <origin xyz="0.116158 -0.170464 -0.0436598" rpy="0.202086 2.47965 0"/>
+      </joint>
+    </xacro:if>
+    <xacro:if value="${wearer_arms == 'down'}">
+      <!-- arms hanging at the sides (the shipped model) -->
+      <link name="human_left_upper_arm">
+        <collision><geometry><cylinder radius="0.05" length="0.3"/></geometry></collision>
+        <visual><geometry><cylinder radius="0.05" length="0.3"/></geometry>
+          <material name="shirt"/></visual>
+      </link>
+      <joint name="torso_to_human_left_upper_arm" type="fixed">
+        <parent link="torso"/><child link="human_left_upper_arm"/>
+        <origin xyz="0.21 0 0.23" rpy="0 3.14159 0"/>
+      </joint>
+      <link name="human_left_lower_arm">
+        <collision><geometry><cylinder radius="0.045" length="0.26"/></geometry></collision>
+        <visual><geometry><cylinder radius="0.045" length="0.26"/></geometry>
+          <material name="skin"/></visual>
+      </link>
+      <joint name="torso_to_human_left_lower_arm" type="fixed">
+        <parent link="torso"/><child link="human_left_lower_arm"/>
+        <origin xyz="0.21 0 -0.05" rpy="0 3.14159 0"/>
+      </joint>
+      <link name="human_left_hand">
+        <collision><geometry><box size="0.09 0.05 0.18"/></geometry></collision>
+        <visual><geometry><box size="0.09 0.05 0.18"/></geometry>
+          <material name="skin"/></visual>
+      </link>
+      <joint name="torso_to_human_left_hand" type="fixed">
+        <parent link="torso"/><child link="human_left_hand"/>
+        <origin xyz="0.21 0 -0.27" rpy="0 3.14159 0"/>
+      </joint>
+      <link name="human_right_upper_arm">
+        <collision><geometry><cylinder radius="0.05" length="0.3"/></geometry></collision>
+        <visual><geometry><cylinder radius="0.05" length="0.3"/></geometry>
+          <material name="shirt"/></visual>
+      </link>
+      <joint name="torso_to_human_right_upper_arm" type="fixed">
+        <parent link="torso"/><child link="human_right_upper_arm"/>
+        <origin xyz="-0.21 0 0.23" rpy="0 -3.14159 0"/>
+      </joint>
+      <link name="human_right_lower_arm">
+        <collision><geometry><cylinder radius="0.045" length="0.26"/></geometry></collision>
+        <visual><geometry><cylinder radius="0.045" length="0.26"/></geometry>
+          <material name="skin"/></visual>
+      </link>
+      <joint name="torso_to_human_right_lower_arm" type="fixed">
+        <parent link="torso"/><child link="human_right_lower_arm"/>
+        <origin xyz="-0.21 0 -0.05" rpy="0 -3.14159 0"/>
+      </joint>
+      <link name="human_right_hand">
+        <collision><geometry><box size="0.09 0.05 0.18"/></geometry></collision>
+        <visual><geometry><box size="0.09 0.05 0.18"/></geometry>
+          <material name="skin"/></visual>
+      </link>
+      <joint name="torso_to_human_right_hand" type="fixed">
+        <parent link="torso"/><child link="human_right_hand"/>
+        <origin xyz="-0.21 0 -0.27" rpy="0 -3.14159 0"/>
+      </joint>
+    </xacro:if>
+    <xacro:if value="${wearer_arms == 'folded'}">
+      <!-- folded across the chest (the forearms are IN the work volume) -->
+      <link name="human_left_upper_arm">
+        <collision><geometry><cylinder radius="0.05" length="0.3"/></geometry></collision>
+        <visual><geometry><cylinder radius="0.05" length="0.3"/></geometry>
+          <material name="shirt"/></visual>
+      </link>
+      <joint name="torso_to_human_left_upper_arm" type="fixed">
+        <parent link="torso"/><child link="human_left_upper_arm"/>
+        <origin xyz="0.217518 0.0270637 0.232653" rpy="-0.181418 3.09062 0"/>
+      </joint>
+      <link name="human_left_lower_arm">
+        <collision><geometry><cylinder radius="0.045" length="0.26"/></geometry></collision>
+        <visual><geometry><cylinder radius="0.045" length="0.26"/></geometry>
+          <material name="skin"/></visual>
+      </link>
+      <joint name="torso_to_human_left_lower_arm" type="fixed">
+        <parent link="torso"/><child link="human_left_lower_arm"/>
+        <origin xyz="0.101566 0.0905183 0.103502" rpy="-0.283721 -1.42448 0"/>
+      </joint>
+      <link name="human_left_hand">
+        <collision><geometry><box size="0.09 0.05 0.18"/></geometry></collision>
+        <visual><geometry><box size="0.09 0.05 0.18"/></geometry>
+          <material name="skin"/></visual>
+      </link>
+      <joint name="torso_to_human_left_hand" type="fixed">
+        <parent link="torso"/><child link="human_left_hand"/>
+        <origin xyz="-0.105478 0.140389 0.152252" rpy="-0.150341 -1.2203 0"/>
+      </joint>
+      <link name="human_right_upper_arm">
+        <collision><geometry><cylinder radius="0.05" length="0.3"/></geometry></collision>
+        <visual><geometry><cylinder radius="0.05" length="0.3"/></geometry>
+          <material name="shirt"/></visual>
+      </link>
+      <joint name="torso_to_human_right_upper_arm" type="fixed">
+        <parent link="torso"/><child link="human_right_upper_arm"/>
+        <origin xyz="-0.217518 0.0270637 0.232653" rpy="-0.181418 -3.09062 0"/>
+      </joint>
+      <link name="human_right_lower_arm">
+        <collision><geometry><cylinder radius="0.045" length="0.26"/></geometry></collision>
+        <visual><geometry><cylinder radius="0.045" length="0.26"/></geometry>
+          <material name="skin"/></visual>
+      </link>
+      <joint name="torso_to_human_right_lower_arm" type="fixed">
+        <parent link="torso"/><child link="human_right_lower_arm"/>
+        <origin xyz="-0.101566 0.0905183 0.103502" rpy="-0.283721 1.42448 0"/>
+      </joint>
+      <link name="human_right_hand">
+        <collision><geometry><box size="0.09 0.05 0.18"/></geometry></collision>
+        <visual><geometry><box size="0.09 0.05 0.18"/></geometry>
+          <material name="skin"/></visual>
+      </link>
+      <joint name="torso_to_human_right_hand" type="fixed">
+        <parent link="torso"/><child link="human_right_hand"/>
+        <origin xyz="0.105478 0.140389 0.152252" rpy="-0.150341 1.2203 0"/>
+      </joint>
+    </xacro:if>
+    <xacro:if value="${wearer_arms == 'none'}">
+      <!-- no wearer arms at all - the limit, not a posture -->
+      <!-- no links: the wearer has no arms in this configuration -->
+    </xacro:if>
+    <xacro:if value="${wearer_arms == 'out'}">
+      <!-- held out to the sides and back, elbows out, hands low and behind -->
+      <link name="human_left_upper_arm">
+        <collision><geometry><cylinder radius="0.05" length="0.3"/></geometry></collision>
+        <visual><geometry><cylinder radius="0.05" length="0.3"/></geometry>
+          <material name="shirt"/></visual>
+      </link>
+      <joint name="torso_to_human_left_upper_arm" type="fixed">
+        <parent link="torso"/><child link="human_left_upper_arm"/>
+        <origin xyz="0.307141 -0.0523068 0.278375" rpy="0.356197 2.37875 0"/>
+      </joint>
+      <link name="human_left_lower_arm">
+        <collision><geometry><cylinder radius="0.045" length="0.26"/></geometry></collision>
+        <visual><geometry><cylinder radius="0.045" length="0.26"/></geometry>
+          <material name="skin"/></visual>
+      </link>
+      <joint name="torso_to_human_left_lower_arm" type="fixed">
+        <parent link="torso"/><child link="human_left_lower_arm"/>
+        <origin xyz="0.497939 -0.169653 0.114313" rpy="0.523946 2.1588 0"/>
+      </joint>
+      <link name="human_left_hand">
+        <collision><geometry><box size="0.09 0.05 0.18"/></geometry></collision>
+        <visual><geometry><box size="0.09 0.05 0.18"/></geometry>
+          <material name="skin"/></visual>
+      </link>
+      <joint name="torso_to_human_left_hand" type="fixed">
+        <parent link="torso"/><child link="human_left_hand"/>
+        <origin xyz="0.654579 -0.28148 0.00778671" rpy="0.546699 2.18152 0"/>
+      </joint>
+      <link name="human_right_upper_arm">
+        <collision><geometry><cylinder radius="0.05" length="0.3"/></geometry></collision>
+        <visual><geometry><cylinder radius="0.05" length="0.3"/></geometry>
+          <material name="shirt"/></visual>
+      </link>
+      <joint name="torso_to_human_right_upper_arm" type="fixed">
+        <parent link="torso"/><child link="human_right_upper_arm"/>
+        <origin xyz="-0.307141 -0.0523068 0.278375" rpy="0.356197 -2.37875 0"/>
+      </joint>
+      <link name="human_right_lower_arm">
+        <collision><geometry><cylinder radius="0.045" length="0.26"/></geometry></collision>
+        <visual><geometry><cylinder radius="0.045" length="0.26"/></geometry>
+          <material name="skin"/></visual>
+      </link>
+      <joint name="torso_to_human_right_lower_arm" type="fixed">
+        <parent link="torso"/><child link="human_right_lower_arm"/>
+        <origin xyz="-0.497939 -0.169653 0.114313" rpy="0.523946 -2.1588 0"/>
+      </joint>
+      <link name="human_right_hand">
+        <collision><geometry><box size="0.09 0.05 0.18"/></geometry></collision>
+        <visual><geometry><box size="0.09 0.05 0.18"/></geometry>
+          <material name="skin"/></visual>
+      </link>
+      <joint name="torso_to_human_right_hand" type="fixed">
+        <parent link="torso"/><child link="human_right_hand"/>
+        <origin xyz="-0.654579 -0.28148 0.00778671" rpy="0.546699 -2.18152 0"/>
+      </joint>
+    </xacro:if>
+    <!-- END GENERATED WEARER ARMS -->
     <!-- ===================== HARNESS =====================
          Shoulder straps, so the pack reads as worn rather than stuck on. -->
