Commit message: Part 1: the centre is shut by the TORSO, not by the wearer's arms
The project's answer to "why can the work not be in the centre" has been the
wearer's own forearm, measured against a mannequin whose arms hang rigidly at
its sides. That is a modelling choice, so the posture is now a variable with
one source and the sweep was re-run in four postures plus the limit case of no
arms at all.

The centre does not open in any of them. With the wearer's arms deleted
entirely, min |x| is still 0.300 (left) and 0.375 (right), every column from
0.125 to 0.300 binds on the TORSO, and at |x| = 0.10 the clearance is -0.007
and -0.013 m, which is the arm inside the person's chest. Holding the arms
clear is worth 25 mm on the left and 75 mm on the right.

Folding the arms across the chest costs 75 mm. Clasping them behind the back
or holding them out to the sides puts the wearer's own limbs inside the
BACK-mounted robot's envelope and breaches the 150 mm floor at the HOME pose,
before anything has been asked of the arm. The useful instruction to a wearer
is "arms down at your sides", which is what the model already assumed and what
nobody had checked was the best of the options.

base_link caps every clearance figure at 0.1610 m. It is a link no joint moves,
so a reading of exactly 0.1610 is the mount's clearance and not the arm's, and
the 150 mm floor has 11 mm of headroom before the arm does anything.

Two live instrument faults found on the way:

  clearance.py, which ik_follower_node, real_homing_node and sim_to_real_bridge
  enforce at runtime, modelled a torso, a head and a pair of hips. The wearer's
  arms were not in it, and they are what binds the right arm inboard, so the
  planner's wearer and the follower's wearer were different people.

  record_verification.py drew the wearer's upper arms 150 mm and forearms
  130 mm below where they are, and omitted the hands.

The published innermost-safe columns are stale. centre_vs_height.json records
0.425 / 0.400; re-running that same script unchanged at z = 1.120 returns
0.325 / 0.450 today, matching the new sweep, because the home change moved the
IK seed and therefore the null-space branch. TASK_SPEC is corrected.

Two of my own controls were wrong and both are recorded in findings.md: a
control whose ground truth moves with the thing under test refused two of the
postures the sweep exists to measure, and a malformed shell line left two
stacks running so one measurement read the wrong robot_description. The URDF
control caught that, which is what it is for.

Tests: 545 pass, 2 allowed failures, 0 new.

This commit also lands the previous session's uncommitted work, which was
never checked in: the predictive-avoidance module and its verification, the
centre-on-surface search, the home storage-site audit and the grasp-approach
measurements.

File: src/srl_description/urdf/srl_dual.urdf.xacro (robot description, xacro)
@@ -47,8 +47,20 @@
   <xacro:include filename="$(find kortex_description)/grippers/robotiq_2f_85/urdf/robotiq_2f_85_macro.xacro"/>
   <!-- LEFT arm.
-       initial_positions == the LEGACY REAL home, so sim and real start at the
-       SAME pose and enabling the sim->real bridge is a no-op rather than a
-       jump. Kortex 259.03/277.69/267.74/286.14/194.10/27.48/55.26.
-       Mirrors config/home_positions_left.txt; keep the two in step. -->
+       initial_positions == THE PRESENTATION POSE (set 2026-08-15), which is
+       now the home pose: wrist level, hand in front of the chest.
+       Kortex 225.18/294.52/333.89/281.93/208.01/321.90/166.67.
+       Mirrors config/home_positions_left.txt; KEEP THE TWO IN STEP.
+       One updated without the other is a documented trap in this project.
+       SIM AND REAL NOW DISAGREE, DELIBERATELY AND TEMPORARILY. The real arm
+       is still parked at the legacy Kortex home
+       259.03/277.69/267.74/286.14/194.10/27.48/55.26, so enabling the
+       sim->real bridge is NOT a no-op any more. It is not a jump either:
+       sim_to_real_bridge.enable() checks the real arm against
+       home_positions_left.txt and REFUSES, naming the joint and the size.
+       The pose is captured on the hardware next lab session (see
+       docs/NEXT_SESSION.md); until then the refusal is the design.
+       This value is baked at LAUNCH, so a colcon build is required before the
+       sim arms start here. Text files changed without a rebuild leave the
+       arms at the old pose while everything else says otherwise. -->
   <xacro:load_arm
       parent="left_mount"
@@ -61,5 +73,5 @@
       gripper_joint_name="left_robotiq_85_left_knuckle_joint"
       use_internal_bus_gripper_comm="true"
-      initial_positions="${dict(joint_1=-1.7623,joint_2=-1.4366,joint_3=-1.6102,joint_4=-1.2891,joint_5=-2.8955,joint_6=0.4796,joint_7=0.9645)}">
+      initial_positions="${dict(joint_1=-2.3530,joint_2=-1.1429,joint_3=-0.4557,joint_4=-1.3626,joint_5=-2.6528,joint_6=-0.6649,joint_7=2.9090)}">
     <origin xyz="0 0 0" rpy="0 0 0"/>
   </xacro:load_arm>
@@ -73,9 +85,15 @@
       moveit_active="true"/>
   <!-- RIGHT arm.
-       initial_positions == the LEGACY REAL home, same reasoning as the left.
-       This gives up the mirror symmetry the previous pose had; matching the
-       real arm matters more, because a mismatch is a commanded jump.
-       Kortex 303.65/77.06/98.57/58.57/317.14/36.39/154.71.
-       Mirrors config/home_positions_right.txt; keep the two in step. -->
+       initial_positions == THE PRESENTATION POSE, same reasoning as the left.
+       Kortex 309.40/100.81/96.22/78.88/11.47/330.88/265.75.
+       Mirrors config/home_positions_right.txt; KEEP THE TWO IN STEP.
+       joint_7 is -1.6450 rad here, NOT the 4.6382 the pose search returned.
+       joint_7 is continuous, so they are the same physical pose, but
+       ik_follower_node refuses to start on real hardware with a continuous
+       joint outside +/-pi and unwinds it in sim. The Kortex value is 265.75
+       either way, so the lab capture is unambiguous.
+       The real arm is still at the legacy Kortex home
+       303.65/77.06/98.57/58.57/317.14/36.39/154.71; the bridge refuses on
+       the difference rather than commanding it. -->
   <xacro:load_arm
       parent="right_mount"
@@ -88,5 +106,5 @@
       gripper_joint_name="right_robotiq_85_left_knuckle_joint"
       use_internal_bus_gripper_comm="true"
-      initial_positions="${dict(joint_1=-0.9835,joint_2=1.3450,joint_3=1.7204,joint_4=1.0222,joint_5=-0.7480,joint_6=0.6351,joint_7=2.7002)}">
+      initial_positions="${dict(joint_1=-0.8831,joint_2=1.7594,joint_3=1.6794,joint_4=1.3767,joint_5=0.2002,joint_6=-0.5082,joint_7=-1.6450)}">
     <origin xyz="0 0 0" rpy="0 0 0"/>
   </xacro:load_arm>
